Commit message: feat: 固定 ELF3 腰部关节

File: HomieRL/legged_gym/resources/robots/elf3_description/urdf/elf3.urdf (robot description, URDF)
Before this commit: robot elf3, 36 links, 35 joints
Joints:
- joint waist_y_joint: axis 0 1 0 -> (none); limit lower=-0.5236 upper=0.5236 effort=90 velocity=20 -> (none); type revolute -> fixed
- joint waist_z_joint: axis 0 0 1 -> (none); limit lower=-2.8798 upper=2.8798 effort=150 velocity=20 -> (none); type revolute -> fixed
